File: PCB/Macropad v3-1.kicad_pcb (KiCad board)
At the start: 2 copper layers, 61.9 x 80.7 mm, 17 parts, among them J1 Conn_01x04_Pin, SW1 SW_Push, SW2 SW_Push, SW3 SW_Push, SW4 SW_Push, SW5 SW_Push, SW6 SW_Push, SW7 RotaryEncoder_Switch, U1 XIAO-RP2040-DIP

Commit message: Fixed Schematics
Connections:
- SW5 pad 2: unconnected-(SW5-Pad2) -> Net-(U1-GPIO0/TX)
- SW6 pad 2: unconnected-(SW6-Pad2) -> Net-(U1-GPIO1/RX)
- U1 pad 7: unconnected-(U1-GPIO0/TX-Pad7) -> Net-(U1-GPIO0/TX)
- U1 pad 8: unconnected-(U1-GPIO1/RX-Pad8) -> Net-(U1-GPIO1/RX)
Routing:
- net Net-(U1-GPIO1/RX): track 0.00 -> 50.8 mm
- net Net-(U1-GPIO0/TX): track 0.00 -> 49.2 mm
Changed lines of the file:
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@@
 	(net 8 "Net-(U1-GPIO4{slash}MISO)")
 	(net 9 "Net-(U1-GPIO3{slash}MOSI)")
-	(net 10 "unconnected-(U1-GPIO0{slash}TX-Pad7)")
+	(net 10 "Net-(U1-GPIO0{slash}TX)")
 	(net 11 "Net-(U1-GPIO27{slash}ADC1{slash}A1)")
 	(net 12 "Net-(U1-GPIO28{slash}ADC2{slash}A2)")
 	(net 13 "Net-(U1-GPIO29{slash}ADC3{slash}A3)")
-	(net 14 "unconnected-(SW5-Pad2)")
-	(net 15 "unconnected-(SW6-Pad2)")
-	(net 16 "unconnected-(U1-GPIO1{slash}RX-Pad8)")
+	(net 14 "Net-(U1-GPIO1{slash}RX)")
 	(footprint "Button_Switch_Keyboard:SW_Cherry_MX_1.00u_PCB"
 		(layer "F.Cu")
@@
 			(layers "*.Cu" "*.Mask")
 			(remove_unused_layers no)
-			(net 15 "unconnected-(SW6-Pad2)")
+			(net 14 "Net-(U1-GPIO1{slash}RX)")
 			(pinfunction "2")
 			(pintype "passive")
@@
 			(layers "*.Cu" "*.Mask")
 			(remove_unused_layers no)
-			(net 14 "unconnected-(SW5-Pad2)")
+			(net 10 "Net-(U1-GPIO0{slash}TX)")
 			(pinfunction "2")
 			(pintype "passive")
@@
 			(layers "F.Cu" "F.Mask")
 			(roundrect_rratio 0.1)
-			(net 10 "unconnected-(U1-GPIO0{slash}TX-Pad7)")
+			(net 10 "Net-(U1-GPIO0{slash}TX)")
 			(pinfunction "GPIO0/TX")
 			(pintype "passive")
@@
 			(layers "*.Cu" "*.Mask")
 			(remove_unused_layers no)
-			(net 10 "unconnected-(U1-GPIO0{slash}TX-Pad7)")
+			(net 10 "Net-(U1-GPIO0{slash}TX)")
 			(pinfunction "GPIO0/TX")
 			(pintype "passive")
@@
 			(layers "*.Cu" "*.Mask")
 			(remove_unused_layers no)
-			(net 16 "unconnected-(U1-GPIO1{slash}RX-Pad8)")
+			(net 14 "Net-(U1-GPIO1{slash}RX)")
 			(pinfunction "GPIO1/RX")
 			(pintype "passive")
@@
 			(layers "F.Cu" "F.Mask")
 			(roundrect_rratio 0.1)
-			(net 16 "unconnected-(U1-GPIO1{slash}RX-Pad8)")
+			(net 14 "Net-(U1-GPIO1{slash}RX)")
 			(pinfunction "GPIO1/RX")
 			(pintype "passive")
@@
 	)
 	(segment
+		(start 67.6275 149.86)
+		(end 69.0285 148.459)
+		(width 0.2)
+		(layer "F.Cu")
+		(net 10)
+	)
+	(segment
+		(start 69.0285 148.459)
+		(end 69.0285 103.4285)
+		(width 0.2)
+		(layer "F.Cu")
+		(net 10)
+	)
+	(segment
+		(start 69.0285 103.4285)
+		(end 67.46 101.86)
+		(width 0.2)
+		(layer "F.Cu")
+		(net 10)
+	)
+	(segment
 		(start 86.6775 111.76)
 		(end 86.6775 108.3775)
@@
 		(net 13)
 	)
+	(segment
+		(start 86.6775 149.86)
+		(end 88.0785 148.459)
+		(width 0.2)
+		(layer "F.Cu")
+		(net 14)
+	)
+	(segment
+		(start 88.0785 107.2385)
+		(end 82.7 101.86)
+		(width 0.2)
+		(layer "F.Cu")
+		(net 14)
+	)
+	(segment
+		(start 88.0785 148.459)
+		(end 88.0785 107.2385)
+		(width 0.2)
+		(layer "F.Cu")
+		(net 14)
+	)
 	(embedded_fonts no)
