File: PCB/Macropad v3-1.kicad_sch (KiCad schematic)
At the start: 9 parts, among them J1 Conn_01x04_Pin, SW1 SW_Push, SW2 SW_Push, SW3 SW_Push, SW4 SW_Push, SW5 SW_Push, SW6 SW_Push, SW7 RotaryEncoder_Switch, U1 XIAO-RP2040-DIP

Commit message: Fixed Schematics
Connections:
- net at SW5.2: now also U1.7 (GPIO0/TX)
- net at SW6.2: now also U1.8 (GPIO1/RX)
Other:
- moved on the sheet: J1, SW1, SW2, SW3, SW4, SW5, SW6, SW7, U1
