File: PCB/Macropad v3-2.kicad_pcb (KiCad board)
At the start: 2 copper layers, 61.9 x 80.7 mm, 17 parts, among them J1 Conn_01x04_Pin, SW1 SW_Push, SW2 SW_Push, SW3 SW_Push, SW4 SW_Push, SW5 SW_Push, SW6 SW_Push, SW7 RotaryEncoder_Switch, U1 XIAO-RP2040-DIP

Commit message: Update Schematics and Case
Connections:
- U1 pad 5: Net-(J1-Pin_3) -> Net-(J1-Pin_4)
- U1 pad 6: Net-(J1-Pin_4) -> Net-(J1-Pin_3)
Routing:
- net Net-(J1-Pin_4): track 51.0 -> 34.9 mm
- net Net-(J1-Pin_3): track 35.9 -> 33.8 mm
Changed lines of the file:
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@@
 			(layers "F.Cu" "F.Mask")
 			(roundrect_rratio 0.1)
-			(net 1 "Net-(J1-Pin_3)")
+			(net 2 "Net-(J1-Pin_4)")
 			(pinfunction "GPIO6/SDA")
 			(pintype "passive")
@@
 			(layers "*.Cu" "*.Mask")
 			(remove_unused_layers no)
-			(net 1 "Net-(J1-Pin_3)")
+			(net 2 "Net-(J1-Pin_4)")
 			(pinfunction "GPIO6/SDA")
 			(pintype "passive")
@@
 			(layers "F.Cu" "F.Mask")
 			(roundrect_rratio 0.1)
-			(net 2 "Net-(J1-Pin_4)")
+			(net 1 "Net-(J1-Pin_3)")
 			(pinfunction "GPIO7/SCL")
 			(pintype "passive")
@@
 			(layers "*.Cu" "*.Mask")
 			(remove_unused_layers no)
-			(net 2 "Net-(J1-Pin_4)")
+			(net 1 "Net-(J1-Pin_3)")
 			(pinfunction "GPIO7/SCL")
 			(pintype "passive")
@@
 	(segment
 		(start 55.989892 125.5)
-		(end 63.075 118.414892)
+		(end 62.475 119.014892)
 		(width 0.2)
 		(layer "F.Cu")
@@
 	)
 	(segment
-		(start 63.075 118.414892)
+		(start 62.475 119.014892)
+		(end 62.475 99.525)
+		(width 0.2)
+		(layer "F.Cu")
+		(net 1)
+	)
+	(via
+		(at 62.475 99.525)
+		(size 0.6)
+		(drill 0.3)
+		(layers "F.Cu" "B.Cu")
+		(net 1)
+	)
+	(segment
+		(start 62.68 99.32)
+		(end 67.46 99.32)
+		(width 0.2)
+		(layer "B.Cu")
+		(net 1)
+	)
+	(segment
+		(start 62.475 99.525)
+		(end 62.68 99.32)
+		(width 0.2)
+		(layer "B.Cu")
+		(net 1)
+	)
+	(segment
+		(start 58.5 125.5)
+		(end 63.075 120.925)
+		(width 0.2)
+		(layer "F.Cu")
+		(net 2)
+	)
+	(segment
+		(start 63.075 120.925)
 		(end 63.075 97)
 		(width 0.2)
 		(layer "F.Cu")
-		(net 1)
+		(net 2)
 	)
 	(via
@@
 		(drill 0.3)
 		(layers "F.Cu" "B.Cu")
-		(net 1)
+		(net 2)
 	)
 	(segment
@@
 		(width 0.2)
 		(layer "B.Cu")
-		(net 1)
+		(net 2)
 	)
 	(segment
@@
 		(width 0.2)
 		(layer "B.Cu")
-		(net 1)
+		(net 2)
 	)
 	(segment
@@
 		(width 0.2)
 		(layer "B.Cu")
-		(net 1)
-	)
-	(segment
-		(start 50.999 123.079)
-		(end 50.999 103.976)
-		(width 0.2)
-		(layer "F.Cu")
-		(net 2)
-	)
-	(segment
-		(start 49.729 126.651)
-		(end 49.729 124.349)
-		(width 0.2)
-		(layer "F.Cu")
-		(net 2)
-	)
-	(segment
-		(start 55.65 99.325)
-		(end 62.275 99.325)
-		(width 0.2)
-		(layer "F.Cu")
-		(net 2)
-	)
-	(segment
-		(start 57.349 126.651)
-		(end 49.729 126.651)
-		(width 0.2)
-		(layer "F.Cu")
-		(net 2)
-	)
-	(segment
-		(start 50.999 103.976)
-		(end 55.65 99.325)
-		(width 0.2)
-		(layer "F.Cu")
-		(net 2)
-	)
-	(segment
-		(start 62.275 99.325)
-		(end 62.475 99.525)
-		(width 0.2)
-		(layer "F.Cu")
-		(net 2)
-	)
-	(segment
-		(start 49.729 124.349)
-		(end 50.999 123.079)
-		(width 0.2)
-		(layer "F.Cu")
-		(net 2)
-	)
-	(segment
-		(start 58.5 125.5)
-		(end 57.349 126.651)
-		(width 0.2)
-		(layer "F.Cu")
-		(net 2)
-	)
-	(via
-		(at 62.475 99.525)
-		(size 0.6)
-		(drill 0.3)
-		(layers "F.Cu" "B.Cu")
-		(net 2)
-	)
-	(segment
-		(start 62.68 99.32)
-		(end 67.46 99.32)
-		(width 0.2)
-		(layer "B.Cu")
-		(net 2)
-	)
-	(segment
-		(start 62.475 99.525)
-		(end 62.68 99.32)
-		(width 0.2)
-		(layer "B.Cu")
