File: PCB/Macropad v3-2.kicad_sch (KiCad schematic)
At the start: 9 parts, among them J1 Conn_01x04_Pin, SW1 SW_Push, SW2 SW_Push, SW3 SW_Push, SW4 SW_Push, SW5 SW_Push, SW6 SW_Push, SW7 RotaryEncoder_Switch, U1 XIAO-RP2040-DIP

Commit message: Update Schematics and Case
Connections:
- net at J1.3 (Pin_3): now also U1.6 (GPIO7/SCL); no longer U1.5 (GPIO6/SDA)
- net at J1.4 (Pin_4): now also U1.5 (GPIO6/SDA); no longer U1.6 (GPIO7/SCL)
Changed lines of the file:
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@@
+	(wire
+		(pts
+			(xy 102.87 168.91) (xy 102.87 182.88)
+		)
+		(stroke
+			(width 0)
+			(type default)
+		)
+	)
 	(wire
 		(pts
@@
 	(wire
 		(pts
+			(xy 90.17 171.45) (xy 100.33 171.45)
+		)
+		(stroke
+			(width 0)
+			(type default)
+		)
+	)
+	(wire
+		(pts
 			(xy 48.26 130.81) (xy 48.26 113.03)
 		)
@@
 	(wire
 		(pts
-			(xy 55.88 120.65) (xy 63.5 120.65)
-		)
-		(stroke
-			(width 0)
-			(type default)
-		)
-	)
-	(wire
-		(pts
 			(xy 90.17 166.37) (xy 102.87 166.37)
 		)
@@
 	(wire
 		(pts
+			(xy 57.15 120.65) (xy 63.5 120.65)
+		)
+		(stroke
+			(width 0)
+			(type default)
+		)
+	)
+	(wire
+		(pts
+			(xy 60.96 182.88) (xy 60.96 124.46)
+		)
+		(stroke
+			(width 0)
+			(type default)
+		)
+	)
+	(wire
+		(pts
+			(xy 90.17 168.91) (xy 102.87 168.91)
+		)
+		(stroke
+			(width 0)
+			(type default)
+		)
+	)
+	(wire
+		(pts
 			(xy 102.87 166.37) (xy 102.87 113.03)
 		)
@@
 	(wire
 		(pts
-			(xy 90.17 168.91) (xy 102.87 168.91)
-		)
-		(stroke
-			(width 0)
-			(type default)
-		)
-	)
-	(wire
-		(pts
 			(xy 35.56 99.06) (xy 30.48 99.06)
 		)
@@
 	(wire
 		(pts
+			(xy 100.33 186.69) (xy 57.15 186.69)
+		)
+		(stroke
+			(width 0)
+			(type default)
+		)
+	)
+	(wire
+		(pts
 			(xy 132.08 140.97) (xy 138.43 140.97)
 		)
@@
 	(wire
 		(pts
-			(xy 90.17 171.45) (xy 100.33 171.45)
-		)
-		(stroke
-			(width 0)
-			(type default)
-		)
-	)
-	(wire
-		(pts
 			(xy 30.48 130.81) (xy 30.48 144.78)
 		)
@@
 	(wire
 		(pts
-			(xy 102.87 186.69) (xy 55.88 186.69)
-		)
-		(stroke
-			(width 0)
-			(type default)
-		)
-	)
-	(wire
-		(pts
-			(xy 102.87 168.91) (xy 102.87 186.69)
+			(xy 102.87 182.88) (xy 60.96 182.88)
+		)
+		(stroke
+			(width 0)
+			(type default)
+		)
+	)
+	(wire
+		(pts
+			(xy 57.15 186.69) (xy 57.15 120.65)
 		)
 		(stroke
@@
 	(wire
 		(pts
-			(xy 59.69 124.46) (xy 63.5 124.46)
+			(xy 60.96 124.46) (xy 63.5 124.46)
 		)
 		(stroke
@@
 	(wire
 		(pts
+			(xy 100.33 171.45) (xy 100.33 186.69)
+		)
+		(stroke
+			(width 0)
+			(type default)
+		)
+	)
+	(wire
+		(pts
 			(xy 63.5 157.48) (xy 63.5 128.27)
 		)
@@
 	(wire
 		(pts
-			(xy 100.33 171.45) (xy 100.33 184.15)
-		)
-		(stroke
-			(width 0)
-			(type default)
-		)
-	)
-	(wire
-		(pts
 			(xy 44.45 115.57) (xy 45.72 115.57)
 		)
@@
 	(wire
 		(pts
-			(xy 59.69 184.15) (xy 59.69 124.46)
-		)
-		(stroke
-			(width 0)
-			(type default)
-		)
-	)
-	(wire
-		(pts
-			(xy 55.88 186.69) (xy 55.88 120.65)
-		)
-		(stroke
-			(width 0)
-			(type default)
-		)
-	)
-	(wire
-		(pts
 			(xy 30.48 170.18) (xy 30.48 175.26)
 		)
 		(stroke
-			(width 0)
-			(type default)
-		)
-	)
-	(wire
-		(pts
-			(xy 100.33 184.15) (xy 59.69 184.15)
-		)
-		(stroke
